File: SO_26_OBC_PCB/so_26_obc_pcb/so_26_obc_pcb.kicad_sch (KiCad schematic)
At the start: 52 parts, among them J1 Conn_02x06_Odd_Even, J2 Conn_02x12_Odd_Even, J3 Conn_01x04, J4 Conn_01x03, J5 Conn_01x02, J6 Conn_01x02, J7 Conn_01x02, J8 Conn_01x03, J9 Conn_01x03, SW1 SW_Push, U1 STM32G431RBTx, U2 TPT3232A-TS3R, U3 PCT2075, U4 MPRLS0025, U5 LSM6DS3, U6 MEM2067-02-180-00-A

Commit message: Latest updates on rev1
Parts:
- removed C11, C12, C14, C15, C8: 100n, Capacitor_SMD:C_0805_2012Metric_Pad1.18x1.45mm_HandSolder, symbol Device:C_Small
- removed J1: Conn_02x06_Odd_Even, Connector_PinSocket_2.54mm:PinSocket_2x06_P2.54mm_Vertical, symbol Connector_Generic:Conn_02x06_Odd_Even
- removed J2: Conn_02x12_Odd_Even, Connector_PinSocket_2.54mm:PinSocket_2x12_P2.54mm_Vertical, symbol Connector_Generic:Conn_02x12_Odd_Even
- removed J3: Conn_01x04, Connector_PinHeader_2.54mm:PinHeader_1x04_P2.54mm_Vertical, symbol Connector_Generic:Conn_01x04
- removed J5, J6, J7: Conn_01x02, Connector_PinSocket_2.54mm:PinSocket_1x02_P2.54mm_Vertical, symbol Connector_Generic:Conn_01x02
- removed J8, J9: Conn_01x03, Connector_PinHeader_2.54mm:PinHeader_1x03_P2.54mm_Vertical, symbol Connector_Generic:Conn_01x03
- removed R7: 10k, Resistor_SMD:R_0805_2012Metric_Pad1.20x1.40mm_HandSolder, symbol Device:R_Small
- removed U2: TPT3232A-TS3R, Package_SO:TSSOP-16_4.4x5mm_P0.65mm, symbol so_26_obc_library:TPT3232A-TS3R
- added C17: 100n, symbol Device:C_Small
- added J1: Conn_02x20_Counter_Clockwise, symbol Connector_Generic:Conn_02x20_Counter_Clockwise
- added J2: Conn_02x06_Top_Bottom, symbol Connector_Generic:Conn_02x06_Top_Bottom
- added J3: Conn_01x03, symbol Connector_Generic:Conn_01x03
- added U6: TPT3232A-TS3R, symbol so_26_obc_library:TPT3232A-TS3R
- C1: renamed from C3; footprint Capacitor_SMD:C_0805_2012Metric_Pad1.18x1.45mm_HandSolder -> (none)
- C10: renamed from C18; footprint Capacitor_SMD:C_0805_2012Metric_Pad1.18x1.45mm_HandSolder -> (none)
- C11: renamed from C20; footprint Capacitor_SMD:C_0805_2012Metric_Pad1.18x1.45mm_HandSolder -> (none)
- C12: renamed from C17; footprint Capacitor_SMD:C_1206_3216Metric_Pad1.33x1.80mm_HandSolder -> (none)
- C13: renamed from C19; footprint Capacitor_SMD:C_0805_2012Metric_Pad1.18x1.45mm_HandSolder -> (none)
- C14: renamed from C21; footprint Capacitor_SMD:C_0805_2012Metric_Pad1.18x1.45mm_HandSolder -> (none)
- C15: renamed from C1; footprint Capacitor_THT:CP_Radial_D6.3mm_P2.50mm -> (none)
- C16: footprint Capacitor_SMD:C_0805_2012Metric_Pad1.18x1.45mm_HandSolder -> (none)
- C2, C7: footprint Capacitor_SMD:C_1206_3216Metric_Pad1.33x1.80mm_HandSolder -> (none)
- C3: renamed from C4; footprint Capacitor_SMD:C_0805_2012Metric_Pad1.18x1.45mm_HandSolder -> (none)
- C4: renamed from C5; footprint Capacitor_SMD:C_0805_2012Metric_Pad1.18x1.45mm_HandSolder -> (none)
- C5: renamed from C6; footprint Capacitor_SMD:C_0805_2012Metric_Pad1.18x1.45mm_HandSolder -> (none)
- C6: renamed from C9; footprint Capacitor_SMD:C_0805_2012Metric_Pad1.18x1.45mm_HandSolder -> (none)
- C8: renamed from C10; footprint Capacitor_SMD:C_0805_2012Metric_Pad1.18x1.45mm_HandSolder -> (none)
- C9: renamed from C13; footprint Capacitor_SMD:C_0805_2012Metric_Pad1.18x1.45mm_HandSolder -> (none)
- D1: renamed from D2; footprint LED_SMD:LED_0805_2012Metric_Pad1.15x1.40mm_HandSolder -> (none)
- D2: renamed from D1; value BLUE -> LED_PWR; footprint LED_SMD:LED_0805_2012Metric_Pad1.15x1.40mm_HandSolder -> (none)
- D3: value YELLOW -> LED_PWR; footprint LED_SMD:LED_0805_2012Metric_Pad1.15x1.40mm_HandSolder -> (none)
- D4: value GREEN -> LED_PWR; footprint LED_SMD:LED_0805_2012Metric_Pad1.15x1.40mm_HandSolder -> (none)
- J4: footprint Connector_PinHeader_2.54mm:PinHeader_1x03_P2.54mm_Vertical -> (none)
- R1: renamed from R6; footprint Resistor_SMD:R_0805_2012Metric_Pad1.20x1.40mm_HandSolder -> (none)
- R10: renamed from R4; value 10k -> 1k; footprint Resistor_SMD:R_0805_2012Metric_Pad1.20x1.40mm_HandSolder -> (none)
- R2: renamed from R5; footprint Resistor_SMD:R_0805_2012Metric_Pad1.20x1.40mm_HandSolder -> (none)
- R3: renamed from R2; value 10k -> 1k; footprint Resistor_SMD:R_0805_2012Metric_Pad1.20x1.40mm_HandSolder -> (none)
- R4: renamed from R11; footprint Resistor_SMD:R_0805_2012Metric_Pad1.20x1.40mm_HandSolder -> (none)
- R5: renamed from R8; footprint Resistor_SMD:R_0805_2012Metric_Pad1.20x1.40mm_HandSolder -> (none)
- R6: renamed from R9; footprint Resistor_SMD:R_0805_2012Metric_Pad1.20x1.40mm_HandSolder -> (none)
- R7: renamed from R10; footprint Resistor_SMD:R_0805_2012Metric_Pad1.20x1.40mm_HandSolder -> (none)
- R8: renamed from R1; value 10k -> 1k; footprint Resistor_SMD:R_0805_2012Metric_Pad1.20x1.40mm_HandSolder -> (none)
- R9: renamed from R3; value 10k -> 1k; footprint Resistor_SMD:R_0805_2012Metric_Pad1.20x1.40mm_HandSolder -> (none)
- SW1: footprint Button_Switch_THT:SW_PUSH_6mm -> (none)
- U2: renamed from U3; footprint Package_SO:TSSOP-8_3x3mm_P0.65mm -> so_26_obc_footprint_library:TSSOP-8_3x3mm_P0.65mm
- U4: renamed from U5; footprint Package_LGA:LGA-14_3x2.5mm_P0.5mm_LayoutBorder3x4y -> so_26_obc_footprint_library:LGA-14_3x2.5mm_P0.5mm_LayoutBorder3x4y
- renumbered U4 to U3, U6 to U5
Connections:
- net +10V: now also J1.38 (Pin_38), J1.39 (Pin_39), J1.40 (Pin_40)
- net +3V3: now also C16.1, C17.1, J1.33 (Pin_33), J1.34 (Pin_34), J2.9 (Pin_9), U6.16 (VCC)
- net ALT_+10V: now also J1.35 (Pin_35), J1.36 (Pin_36), J1.37 (Pin_37), J2.7 (Pin_7), J2.8 (Pin_8)
- net GND: now also C16.2, C17.2, J1.1 (Pin_1), J1.10 (Pin_10), J1.11 (Pin_11), J1.12 (Pin_12), J1.13 (Pin_13), J1.14 (Pin_14), J1.15 (Pin_15), J1.16 (Pin_16), J1.17 (Pin_17), J1.18 (Pin_18), J1.19 (Pin_19), J1.2 (Pin_2), J1.20 (Pin_20), J1.3 (Pin_3), J1.4 (Pin_4), J1.5 (Pin_5), J1.6 (Pin_6), J1.7 (Pin_7), J1.8 (Pin_8), J1.9 (Pin_9), J2.1 (Pin_1), J2.2 (Pin_2), J2.3 (Pin_3), J2.4 (Pin_4), J2.5 (Pin_5), J2.6 (Pin_6), J3.2 (Pin_2), U6.15 (GND); no longer C16.1
- net I2C_SDA: now also J2.12 (Pin_12)
- net PWM_HEATER: now also J2.10 (Pin_10)
- net RADIO_UART_RX: now also J1.31 (Pin_31)
- net RADIO_UART_TX: now also J1.32 (Pin_32)
- net SD_MISO: now also R6.1, U5.3 (MOSI); no longer R5.1, U5.7 (MISO)
- net SD_MOSI: now also R5.1, U5.7 (MISO); no longer R6.1, U5.3 (MOSI)
- net SWCLK: now also J3.1 (Pin_1)
- net SWDIO: now also J3.3 (Pin_3)
- net VBAT_0: now also J1.30 (Pin_30)
- net VBAT_1: now also J1.29 (Pin_29)
- net BOOT0 renamed I2C_SCL
- net I2C_SCL: now also J2.11 (Pin_11)
- net LED_BLUE renamed DEBUG_LED_0
- net LED_GREEN renamed DEBUG_LED_2
- net LED_YELLOW renamed DEBUG_LED_1
- net LOW_POWER_MODE: no longer names the net of U1.43 (PA9)
- no-connect marks 46 -> 53
Other:
- note added: "Level shifter for radio"
- note removed: "Debug av kode"
- note removed: "UART-RS232"
- moved on the sheet: C1, C10, C11, C12, C13, C14, C15, C2, C3, C4, C5, C9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
