File: so_26_obc_pcb/so_26_obc_pcb.kicad_sch (KiCad schematic)
At the start: 52 parts, among them J1 Conn_02x06_Odd_Even, J2 Conn_02x12_Odd_Even, J3 Conn_01x04, J4 Conn_01x03, J5 Conn_01x02, J6 Conn_01x02, J7 Conn_01x02, J8 Conn_01x03, J9 Conn_01x03, SW1 SW_Push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

Commit message: PCB: did some routing, almost done
Parts:
- removed J9: Conn_01x03, Connector_PinHeader_2.54mm:PinHeader_1x03_P2.54mm_Vertical, symbol Connector_Generic:Conn_01x03
- added J10: Conn_01x04, Connector_PinHeader_2.54mm:PinHeader_1x04_P2.54mm_Vertical, symbol Connector_Generic:Conn_01x04
Connections:
- net +3V3: now also J10.1 (Pin_1)
- net BOOT0: now also J10.4 (Pin_4)
- net GND: now also J10.3 (Pin_3)
- net I2C_SDA: now also J10.2 (Pin_2)
Other:
- moved on the sheet: J8
Changed lines of the file:
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@@
 	(wire
 		(pts
-			(xy 138.43 177.8) (xy 138.43 176.53)
+			(xy 138.43 175.26) (xy 138.43 173.99)
 		)
 		(stroke
@@
 	(wire
 		(pts
-			(xy 140.97 179.07) (xy 156.21 179.07)
+			(xy 140.97 176.53) (xy 156.21 176.53)
 		)
 		(stroke
@@
 	(wire
 		(pts
-			(xy 148.59 185.42) (xy 156.21 185.42)
+			(xy 148.59 187.96) (xy 156.21 187.96)
 		)
 		(stroke
@@
 	(wire
 		(pts
-			(xy 148.59 190.5) (xy 156.21 190.5)
+			(xy 148.59 193.04) (xy 156.21 193.04)
 		)
 		(stroke
@@
 	(wire
 		(pts
-			(xy 140.97 173.99) (xy 156.21 173.99)
+			(xy 140.97 171.45) (xy 156.21 171.45)
 		)
 		(stroke
@@
 	(wire
 		(pts
-			(xy 146.05 187.96) (xy 156.21 187.96)
+			(xy 146.05 190.5) (xy 156.21 190.5)
 		)
 		(stroke
@@
 	(wire
 		(pts
-			(xy 146.05 189.23) (xy 146.05 187.96)
+			(xy 146.05 190.5) (xy 146.05 191.77)
 		)
 		(stroke
@@
 	(wire
 		(pts
+			(xy 154.94 185.42) (xy 156.21 185.42)
+		)
+		(stroke
+			(width 0)
+			(type default)
+		)
+	)
+	(wire
+		(pts
 			(xy 256.54 140.97) (xy 256.54 142.24)
 		)
@@
 	(wire
 		(pts
+			(xy 154.94 184.15) (xy 154.94 185.42)
+		)
+		(stroke
+			(width 0)
+			(type default)
+		)
+	)
+	(wire
+		(pts
 			(xy 74.93 53.34) (xy 74.93 54.61)
 		)
@@
 	(wire
 		(pts
-			(xy 138.43 176.53) (xy 156.21 176.53)
+			(xy 138.43 173.99) (xy 156.21 173.99)
 		)
 		(stroke
@@
 	)
 	(label "RADIO_UART_RX"
-		(at 140.97 173.99 0)
+		(at 140.97 171.45 0)
 		(fields_autoplaced yes)
 		(effects
@@
 		)
 		(property "Netclass" ""
-			(at 140.97 175.26 0)
+			(at 140.97 172.72 0)
 			(effects
 				(font
@@
 	)
 	(label "RADIO_UART_TX"
-		(at 140.97 179.07 0)
+		(at 140.97 176.53 0)
 		(fields_autoplaced yes)
 		(effects
@@
 		)
 		(property "Netclass" ""
-			(at 140.97 180.34 0)
+			(at 140.97 177.8 0)
 			(effects
 				(font
@@
 	)
 	(label "I2C_SDA"
-		(at 148.59 185.42 0)
+		(at 148.59 187.96 0)
 		(effects
 			(font
@@
 	)
 	(label "I2C_SCL"
-		(at 148.59 190.5 0)
+		(at 148.59 193.04 0)
 		(effects
 			(font
@@
 	)
 	(symbol
+		(lib_id "Connector_Generic:Conn_01x04")
+		(at 161.29 187.96 0)
+		(unit 1)
+		(exclude_from_sim no)
+		(in_bom yes)
+		(on_board yes)
+		(dnp no)
+		(fields_autoplaced yes)
+		(property "Reference" "J10"
+			(at 163.83 187.9599 0)
+			(effects
+				(font
+					(size 1.27 1.27)
+				)
+				(justify left)
+			)
+		)
+		(property "Value" "Conn_01x04"
+			(at 163.83 190.4999 0)
+			(effects
+				(font
+					(size 1.27 1.27)
+				)
+				(justify left)
+			)
+		)
+		(property "Footprint" "Connector_PinHeader_2.54mm:PinHeader_1x04_P2.54mm_Vertical"
+			(at 161.29 187.96 0)
+			(effects
+				(font
+					(size 1.27 1.27)
+				)
+				(hide yes)
+			)
+		)
+		(property "Datasheet" "~"
+			(at 161.29 187.96 0)
+			(effects
+				(font
+					(size 1.27 1.27)
+				)
+				(hide yes)
+			)
+		)
+		(property "Description" "Generic connector, single row, 01x04, script generated (kicad-library-utils/schlib/autogen/connector/)"
+			(at 161.29 187.96 0)
+			(effects
+				(font
+					(size 1.27 1.27)
+				)
+				(hide yes)
+			)
+		)
+		(pin "2"
+		)
+		(pin "3"
+		)
+		(pin "4"
+		)
+		(pin "1"
+		)
+		(instances
+			(project ""
+				(path "/19e03f49-67e8-4e0c-a53b-de9e8097c0a8"
+					(reference "J10")
+					(unit 1)
+				)
+			)
+		)
+	)
+	(symbol
 		(lib_id "Connector_Generic:Conn_02x06_Odd_Even")
 		(at 35.56 168.91 0)
@@
 	(symbol
 		(lib_id "power:GND")
-		(at 138.43 177.8 0)
+		(at 138.43 175.26 0)
 		(unit 1)
 		(exclude_from_sim no)
@@
 		(fields_autoplaced yes)
 		(property "Reference" "#PWR022"
-			(at 138.43 184.15 0)
+			(at 138.43 181.61 0)
 			(effects
 				(font
@@
 		)
 		(property "Value" "GND"
-			(at 138.43 182.88 0)
+			(at 138.43 180.34 0)
 			(effects
 				(font
@@
 		)
 		(property "Footprint" ""
-			(at 138.43 177.8 0)
+			(at 138.43 175.26 0)
 			(effects
 				(font
@@
 		)
 		(property "Datasheet" ""
-			(at 138.43 177.8 0)
+			(at 138.43 175.26 0)
 			(effects
 				(font
@@
 		)
 		(property "Description" "Power symbol creates a global label with name \"GND\" , ground"
-			(at 138.43 177.8 0)
+			(at 138.43 175.26 0)
 			(effects
 				(font
@@
 	(symbol
 		(lib_id "power:GND")
-		(at 146.05 189.23 0)
+		(at 146.05 191.77 0)
 		(unit 1)
 		(exclude_from_sim no)
@@
 		(fields_autoplaced yes)
 		(property "Reference" "#PWR023"
-			(at 146.05 195.58 0)
+			(at 146.05 198.12 0)
 			(effects
 				(font
@@
 		)
 		(property "Value" "GND"
-			(at 146.05 194.31 0)
+			(at 146.05 196.85 0)
 			(effects
 				(font
@@
 		)
 		(property "Footprint" ""
-			(at 146.05 189.23 0)
+			(at 146.05 191.77 0)
 			(effects
 				(font
@@
 		)
 		(property "Datasheet" ""
-			(at 146.05 189.23 0)
+			(at 146.05 191.77 0)
 			(effects
 				(font
@@
 		)
 		(property "Description" "Power symbol creates a global label with name \"GND\" , ground"
-			(at 146.05 189.23 0)
+			(at 146.05 191.77 0)
 			(effects
 				(font
@@
 	(symbol
 		(lib_id "Connector_Generic:Conn_01x03")
-		(at 161.29 176.53 0)
+		(at 161.29 173.99 0)
 		(unit 1)
 		(exclude_from_sim no)
@@
 		(fields_autoplaced yes)
 		(property "Reference" "J8"
-			(at 163.83 175.2599 0)
+			(at 163.83 172.7199 0)
 			(effects
 				(font
@@
 		)
 		(property "Value" "Conn_01x03"
-			(at 163.83 177.7999 0)
+			(at 163.83 175.2599 0)
 			(effects
 				(font
@@
 		)
 		(property "Footprint" "Connector_PinHeader_2.54mm:PinHeader_1x03_P2.54mm_Vertical"
-			(at 161.29 176.53 0)
+			(at 161.29 173.99 0)
 			(effects
 				(font
@@
 		)
 		(property "Datasheet" "~"
-			(at 161.29 176.53 0)
+			(at 161.29 173.99 0)
 			(effects
 				(font
@@
 		)
 		(property "Description" "Generic connector, single row, 01x03, script generated (kicad-library-utils/schlib/autogen/connector/)"
-			(at 161.29 176.53 0)
+			(at 161.29 173.99 0)
 			(effects
 				(font
@@
 	)
 	(symbol
-		(lib_id "Connector_Generic:Conn_01x03")
-		(at 161.29 187.96 0)
-		(unit 1)
-		(exclude_from_sim no)
-		(in_bom yes)
-		(on_board yes)
-		(dnp no)
-		(fields_autoplaced yes)
-		(property "Reference" "J9"
-			(at 163.83 186.6899 0)
-			(effects
-				(font
-					(size 1.27 1.27)
-				)
-				(justify left)
-			)
-		)
-		(property "Value" "Conn_01x03"
-			(at 163.83 189.2299 0)
-			(effects
-				(font
-					(size 1.27 1.27)
-				)
-				(justify left)
-				(hide yes)
-			)
-		)
-		(property "Footprint" "Connector_PinHeader_2.54mm:PinHeader_1x03_P2.54mm_Vertical"
-			(at 161.29 187.96 0)
-			(effects
-				(font
-					(size 1.27 1.27)
-				)
-				(hide yes)
-			)
-		)
-		(property "Datasheet" "~"
-			(at 161.29 187.96 0)
-			(effects
-				(font
-					(size 1.27 1.27)
-				)
-				(hide yes)
-			)
-		)
-		(property "Description" "Generic connector, single row, 01x03, script generated (kicad-library-utils/schlib/autogen/connector/)"
-			(at 161.29 187.96 0)
-			(effects
-				(font
-					(size 1.27 1.27)
-				)
-				(hide yes)
-			)
-		)
-		(pin "1"
-		)
-		(pin "3"
-		)
-		(pin "2"
-		)
-		(instances
-			(project "so_26_obc_pcb"
-				(path "/19e03f49-67e8-4e0c-a53b-de9e8097c0a8"
-					(reference "J9")
-					(unit 1)
-				)
-			)
-		)
-	)
-	(symbol
 		(lib_id "Device:R_Small")
 		(at 26.67 137.16 180)
@@
 					(unit 1)
 				)
+			)
+		)
+	)
+	(symbol
+		(lib_id "power:+3V3")
+		(at 154.94 184.15 0)
+		(unit 1)
+		(exclude_from_sim no)
+		(in_bom yes)
+		(on_board yes)
+		(dnp no)
+		(property "Reference" "#PWR048"
+			(at 154.94 187.96 0)
+			(effects
+				(font
+					(size 1.27 1.27)
+				)
+				(hide yes)
+			)
+		)
+		(property "Value" "+3V3"
+			(at 154.94 180.594 0)
+			(effects
+				(font
+					(size 1.27 1.27)
+				)
+			)
+		)
+		(property "Footprint" ""
+			(at 154.94 184.15 0)
+			(effects
+				(font
+					(size 1.27 1.27)
+				)
+				(hide yes)
+			)
+		)
+		(property "Datasheet" ""
+			(at 154.94 184.15 0)
+			(effects
+				(font
+					(size 1.27 1.27)
+				)
+				(hide yes)
+			)
+		)
+		(property "Description" "Power symbol creates a global label with name \"+3V3\""
+			(at 154.94 184.15 0)
+			(effects
+				(font
+					(size 1.27 1.27)
+				)
+				(hide yes)
+			)
+		)
+		(pin "1"
+		)
+		(instances
+			(project "so_26_obc_pcb"
+				(path "/19e03f49-67e8-4e0c-a53b-de9e8097c0a8"
+					(reference "#PWR048")
+					(unit 1)
+				)
